File: PCB_Frackstock/Frackstock.kicad_pcb (KiCad board)
At the start: 4 copper layers, 23 x 79 mm, 90 parts, among them IC1 DW01A, J1 87224-3, J10 SWD, J2 105450-0101, J5 Conn_01x02_Male, J6 Conn_01x02_Male, J8 Conn_01x02_Male, Q1 FS8205A, Q2 BSS138, U1 RP2040, U10 DFLS130L-7, U11 CC1101RGPR, U12 SPX3819M5-L-3-3, U13 SGM6603-5.0YN6G_TR, U14 1043, U2 W25Q128JVSIQ, U7 BMI160, U8 TP4056, U9 AO3401, Y1 TAXM12M4RLBDDT2T, Y2 JGHC S3226000151040

Commit message: Schema fertig
Parts:
- removed ANT1: W3000, KiCad:W3000
- removed C34: 220p, Capacitor_SMD:C_0201_0603Metric
- removed C35, C36: 10u, Capacitor_SMD:C_0402_1005Metric
- removed IC1: DW01A, SnapEDA Library:SOT23-6
- removed J5: Conn_01x02_Male, Connector_PinHeader_2.54mm:PinHeader_1x02_P2.54mm_Vertical
- removed L2, L3, L5: 27n, Inductor_SMD:L_0201_0603Metric
- removed L4: 22n, Inductor_SMD:L_0201_0603Metric
- removed L6: 3.9n, KiCad:MHQ1005
- removed L7: 27n, KiCad:MLG1005
- removed Q1: FS8205A, SnapEDA Library:SOP65P640X120-8N
- removed Q2: BSS138, Package_TO_SOT_SMD:SOT-23
- removed R17: 10k, Resistor_SMD:R_0201_0603Metric
- removed R21: 100, Resistor_SMD:R_0201_0603Metric
- removed U10: DFLS130L-7, SnapEDA Library:POWERDI123
- removed U13: SGM6603-5.0YN6G_TR, SnapEDA Library:SOT23-6
- removed U8: TP4056, SnapEDA Library:SOP127P600X175-9N
- removed U9: AO3401, SnapEDA Library:SOT23
- removed Y1: TAXM12M4RLBDDT2T, Crystal:Crystal_SMD_3225-4Pin_3.2x2.5mm
- added ANT2: W3000, RF_Antenna:W3000, F.Cu at (45.0, 105.7)
- added C37: 1.5pF, Capacitor_SMD:C_0603_1608Metric_Pad1.08x0.95mm_HandSolder, F.Cu at (25.7, 55.6)
- added C38: 1p, Capacitor_SMD:C_0603_1608Metric_Pad1.08x0.95mm_HandSolder, F.Cu at (30.0, 43.0)
- added C39: 100pF, Capacitor_SMD:C_0603_1608Metric_Pad1.08x0.95mm_HandSolder, F.Cu at (30.0, 45.6)
- added C40: 3.3pF, Capacitor_SMD:C_0603_1608Metric_Pad1.08x0.95mm_HandSolder, F.Cu at (30.0, 48.1)
- added C41: 1.5pF, Capacitor_SMD:C_0603_1608Metric_Pad1.08x0.95mm_HandSolder, F.Cu at (30.0, 50.6)
- added D6: LED, LED_SMD:LED_0603_1608Metric_Pad1.05x0.95mm_HandSolder, F.Cu at (53.8, 67.8)
- added D7: LED, LED_SMD:LED_0603_1608Metric_Pad1.05x0.95mm_HandSolder, F.Cu at (53.8, 70.3)
- added L10: 18nH, Inductor_SMD:L_0603_1608Metric_Pad1.05x0.95mm_HandSolder, F.Cu at (34.4, 43.0)
- added L11: 18nH, Inductor_SMD:L_0603_1608Metric_Pad1.05x0.95mm_HandSolder, F.Cu at (34.4, 45.6)
- added L12: 12nH, Inductor_SMD:L_0603_1608Metric_Pad1.05x0.95mm_HandSolder, F.Cu at (34.4, 48.1)
- added L13: 12nH, Inductor_SMD:L_0603_1608Metric_Pad1.05x0.95mm_HandSolder, F.Cu at (34.4, 50.6)
- added L8: 12nH, Inductor_SMD:L_0603_1608Metric_Pad1.05x0.95mm_HandSolder, F.Cu at (30.0, 53.1)
- added L9: 12nH, Inductor_SMD:L_0603_1608Metric_Pad1.05x0.95mm_HandSolder, F.Cu at (30.0, 55.6)
- added R18: 100, Resistor_SMD:R_0603_1608Metric_Pad0.98x0.95mm_HandSolder, F.Cu at (49.4, 53.1)
- added U3: MCP73871-2CC, Package_DFN_QFN:QFN-20-1EP_4x4mm_P0.5mm_EP2.5x2.5mm, F.Cu at (21.1, 96.8)
- added U4: TPS61222DCK, Package_TO_SOT_SMD:Texas_R-PDSO-G6, F.Cu at (41.1, 121.0)
- added Y3: 12MHz, Crystal:Crystal_SMD_5032-2Pin_5.0x3.2mm, F.Cu at (44.4, 115.5)
- C1, C2: footprint Capacitor_SMD:C_0402_1005Metric -> Capacitor_SMD:C_0603_1608Metric_Pad1.08x0.95mm_HandSolder
- C10, C11, C12, C13, C14, C15, C16, C17, C18, C19, C20, C21, C25, C27, C6, C7, C8, C9: footprint Capacitor_SMD:C_0201_0603Metric -> Capacitor_SMD:C_0603_1608Metric_Pad1.08x0.95mm_HandSolder
- C22, C30: value 25p -> 20p; footprint Capacitor_SMD:C_0402_1005Metric -> Capacitor_SMD:C_0603_1608Metric_Pad1.08x0.95mm_HandSolder
- C23, C26: value 3.9p -> 100n; footprint Capacitor_SMD:C_0201_0603Metric -> Capacitor_SMD:C_0603_1608Metric_Pad1.08x0.95mm_HandSolder
- C24: value 220p -> 100n; footprint Capacitor_SMD:C_0201_0603Metric -> Capacitor_SMD:C_0603_1608Metric_Pad1.08x0.95mm_HandSolder
- C28: value 100n -> 4.7u; footprint Capacitor_SMD:C_0201_0603Metric -> Capacitor_SMD:C_0603_1608Metric_Pad1.08x0.95mm_HandSolder
- C29: value 8.2p -> 4.7u; footprint Capacitor_SMD:C_0201_0603Metric -> Capacitor_SMD:C_0603_1608Metric_Pad1.08x0.95mm_HandSolder
- C3, C31: value 100n -> 10u; footprint Capacitor_SMD:C_0201_0603Metric -> Capacitor_SMD:C_0603_1608Metric_Pad1.08x0.95mm_HandSolder
- C32: value 5.6p -> 10u; footprint Capacitor_SMD:C_0201_0603Metric -> Capacitor_SMD:C_0603_1608Metric_Pad1.08x0.95mm_HandSolder
- C33: value 100n -> 1000u; footprint Capacitor_SMD:C_0201_0603Metric -> Capacitor_SMD:CP_Elec_8x10.5
- C4, C5: value 30q -> 14p; footprint Capacitor_SMD:C_0201_0603Metric -> Capacitor_SMD:C_0603_1608Metric_Pad1.08x0.95mm_HandSolder
- D1: value STDBY -> SMAJ5.0A; footprint LED_SMD:LED_0402_1005Metric -> Diode_SMD:D_SMA
- D2: value CHRG -> LED; footprint LED_SMD:LED_0402_1005Metric -> LED_SMD:LED_0603_1608Metric_Pad1.05x0.95mm_HandSolder
- D3, D4, D5: footprint LED_SMD:LED_0402_1005Metric -> LED_SMD:LED_0603_1608Metric_Pad1.05x0.95mm_HandSolder
- R1, R10, R11, R12, R13, R14, R15, R2, R20, R22, R9: footprint Resistor_SMD:R_0201_0603Metric -> Resistor_SMD:R_0603_1608Metric_Pad0.98x0.95mm_HandSolder
- R16: value 10k -> 470; footprint Resistor_SMD:R_0201_0603Metric -> Resistor_SMD:R_0603_1608Metric_Pad0.98x0.95mm_HandSolder
- R3: value 5.1k -> 2k; footprint Resistor_SMD:R_0201_0603Metric -> Resistor_SMD:R_0603_1608Metric_Pad0.98x0.95mm_HandSolder
- R4: value 330 -> 8k; footprint Resistor_SMD:R_0201_0603Metric -> Resistor_SMD:R_0603_1608Metric_Pad0.98x0.95mm_HandSolder
- R5: value 330 -> 10k; footprint Resistor_SMD:R_0201_0603Metric -> Resistor_SMD:R_0603_1608Metric_Pad0.98x0.95mm_HandSolder
- R6: value 100 -> 330; footprint Resistor_SMD:R_0201_0603Metric -> Resistor_SMD:R_0603_1608Metric_Pad0.98x0.95mm_HandSolder
- R7: value 1k -> 330; footprint Resistor_SMD:R_0201_0603Metric -> Resistor_SMD:R_0603_1608Metric_Pad0.98x0.95mm_HandSolder
- R8: value 1M -> 330; footprint Resistor_SMD:R_0201_0603Metric -> Resistor_SMD:R_0603_1608Metric_Pad0.98x0.95mm_HandSolder
- U12: value SPX3819M5-L-3-3 -> SPX3819M5-L-3-3/TR
- U7: value BMI160 -> BMI323
- Y2: value JGHC S3226000151040 -> 26MHz; footprint Crystal:Crystal_SMD_3225-4Pin_3.2x2.5mm -> Crystal:Crystal_SMD_Abracon_ABM3B-4Pin_5.0x3.2mm
- moved U12 106.6 mm to (42.1, 126.4)
- moved C20 94.5 mm to (21.3, 48.1)
- moved C22 94.0 mm to (21.3, 53.1)
- moved J2 93.2 mm to (26.8, 108.6)
- moved C21 92.6 mm to (21.3, 50.6)
- moved C30 92.5 mm to (25.7, 53.1), turned to 0 degrees
- moved C25 92.2 mm to (25.7, 45.6)
- moved C24 89.9 mm to (25.7, 43.0), turned to 0 degrees
- moved C23 89.8 mm to (21.3, 55.6), turned to 0 degrees
- moved J6 87.1 mm to (28.4, 120.8)
- moved C26 86.7 mm to (25.7, 48.1)
- moved C27 83.3 mm to (25.7, 50.6), turned to 0 degrees
- moved C18 82.6 mm to (21.3, 43.0), turned to 0 degrees
- moved C19 81.8 mm to (21.3, 45.6), turned to 0 degrees
- moved C33 80.0 mm to (25.8, 61.9), turned to 0 degrees
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Connections:
- C23 pad 1: RF_N -> +3.3V
- C24 pad 1: Net-(C24-Pad1) -> +3.3V
- C26 pad 1: RF_P -> +3.3V
- C26 pad 2: Net-(C26-Pad2) -> GND
- C28 pad 1: +3.3V -> GND
- C28 pad 2: GND -> BAT_O
- C29 pad 1: Net-(C29-Pad1) -> GND
- C29 pad 2: GND -> BAT_P
- C3 pad 1: BAT_N -> VBUS
- C3 pad 2: Net-(IC1-VCC) -> GND
- C31 pad 1: +3.3V -> +5V
- C32 pad 1: Net-(C32-Pad1) -> BAT_O
- C33 pad 1: +3.3V -> GND
- C33 pad 2: GND -> BAT_O
- D1 pad 1: STDBY -> VBUS
- D1 pad 2: Net-(D1-A) -> GND
- D2 pad 1: CHRG -> Net-(D2-K)
- D2 pad 2: Net-(D2-A) -> VBUS
- D3 pad 2: LED1 -> LED2
- D4 pad 2: LED2 -> LED1
- J1 pad 1: +5V -> BAT_O
- J1 pad 2: Net-(Q2-D) -> Net-(J1-Pad2)
- R16 pad 1: +3.3V -> LED_DI
- R16 pad 2: LED_DI -> Net-(J1-Pad2)
- R4 pad 1: Net-(D1-A) -> GND
- R4 pad 2: VBUS -> Net-(U3-PROG3)
- R5 pad 1: Net-(D2-A) -> GND
- R5 pad 2: VBUS -> Net-(U3-THERM)
- R6 pad 1: Net-(IC1-VCC) -> Net-(D2-K)
- R6 pad 2: BAT_P -> Net-(U3-~{PG})
- R7 pad 2: GND -> Net-(U3-STAT1/~{LBO})
- R8 pad 1: VBUS -> Net-(D7-K)
- R8 pad 2: GND -> Net-(U3-STAT2)
- R9 pad 1: DN -> Net-(U1-USB_DM)
- R9 pad 2: Net-(U1-USB_DM) -> DN
- U14 pad 2: BAT_N -> GND
Routing:
- net BAT_N: track 89.3 -> 0.00 mm, vias 1 -> 0
- net +3.3V: track 52.5 -> 0.00 mm, vias 17 -> 0
- net VBUS: track 47.4 -> 0.00 mm, vias 4 -> 0
- net BAT_O: track 37.1 -> 0.00 mm, vias 1 -> 0
- net +5V: track 28.1 -> 0.00 mm, vias 2 -> 0
- net unconnected-(ANT1-GND-Pad2): track 25.8 -> 0.00 mm
- net BAT_P: track 25.7 -> 0.00 mm
- net Net-(Q2-D): track 18.6 -> 0.00 mm
- net DP: track 18.3 -> 0.00 mm, vias 3 -> 0
- net SWD: track 17.7 -> 0.00 mm, vias 2 -> 0
- net DN: track 17.1 -> 0.00 mm, vias 3 -> 0
- net SWCLK: track 16.9 -> 0.00 mm, vias 2 -> 0
- net +1V1: track 16.4 -> 0.00 mm, vias 3 -> 0
- net XIN: track 15.6 -> 0.00 mm, vias 2 -> 0
- net XOSC_Q2: track 15.5 -> 0.00 mm, vias 2 -> 0
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- removed copper zone on F.Cu, net +1V1
Other:
- board size 23 x 79 mm -> 23 x 100 mm

Commit message: Schema_fertig
Parts:
- removed C1, C2, C31, C32: 10u, Capacitor_SMD:C_0603_1608Metric_Pad1.08x0.95mm_HandSolder
- removed C10, C11, C12, C13, C14, C15, C16, C17, C6, C7: 100n, Capacitor_SMD:C_0603_1608Metric_Pad1.08x0.95mm_HandSolder
- removed C4, C5: 14p, Capacitor_SMD:C_0603_1608Metric_Pad1.08x0.95mm_HandSolder
- removed C8, C9: 1u, Capacitor_SMD:C_0603_1608Metric_Pad1.08x0.95mm_HandSolder
- removed D3, D4, D5: LED, LED_SMD:LED_0603_1608Metric_Pad1.05x0.95mm_HandSolder
- removed J10: SWD, SnapEDA Library:JST_SM03B-SRSS-TB(LF)(SN)
- removed L1: 4.7u, Inductor_SMD:L_0603_1608Metric
- removed R10, R9: 27.4, Resistor_SMD:R_0603_1608Metric_Pad0.98x0.95mm_HandSolder
- removed R11: 1k, Resistor_SMD:R_0603_1608Metric_Pad0.98x0.95mm_HandSolder
- removed R12: 10k, Resistor_SMD:R_0603_1608Metric_Pad0.98x0.95mm_HandSolder
- removed R14, R15, R22: 330, Resistor_SMD:R_0603_1608Metric_Pad0.98x0.95mm_HandSolder
- removed R18, R20: 100, Resistor_SMD:R_0603_1608Metric_Pad0.98x0.95mm_HandSolder
- removed U12: SPX3819M5-L-3-3/TR, Package_TO_SOT_SMD:SOT-23-5
- removed U2: W25Q128JVSIQ, SnapEDA Library:SOIC127P790X216-8N
- removed U4: TPS61222DCK, Package_TO_SOT_SMD:Texas_R-PDSO-G6
- removed Y3: 12MHz, Crystal:Crystal_SMD_5032-2Pin_5.0x3.2mm
- added J3: Conn_01x03_Pin, Connector_PinHeader_2.54mm:PinHeader_1x03_P2.54mm_Vertical, F.Cu at (94.7, 57.7)
- added J4: Conn_01x02_Male, Connector_PinHeader_2.54mm:PinHeader_1x02_P2.54mm_Vertical, F.Cu at (82.0, 58.8)
- added J5: Conn_01x02_Pin, Connector_PinHeader_2.54mm:PinHeader_1x02_P2.54mm_Vertical, F.Cu at (72.7, 58.8)
- added J7: Conn_01x04_Pin, Connector_PinHeader_2.54mm:PinHeader_1x04_P2.54mm_Vertical, F.Cu at (90.1, 57.7)
- added JP1: SolderJumper_2_Open, Jumper:SolderJumper-2_P1.3mm_Open_RoundedPad1.0x1.5mm, F.Cu at (140.2, 60.3)
- added TP1: TestPoint_Alt, TestPoint:TestPoint_Pad_1.5x1.5mm, F.Cu at (130.0, 75.0)
- added TP2: TestPoint_Alt, TestPoint:TestPoint_Pad_1.5x1.5mm, F.Cu at (132.0, 75.0)
- added TP3: TestPoint_Alt, TestPoint:TestPoint_Pad_1.5x1.5mm, F.Cu at (128.4, 74.9)
- C20, C21, C22, C23, C24, C25, C26, C27, C30, R13, U11, Y2: moved to B.Cu
- J1: value 87224-3 -> Conn_01x03_Pin; footprint KiCad:872243 -> Connector_PinHeader_2.54mm:PinHeader_1x03_P2.54mm_Vertical
- J6: value Conn_01x02_Male -> Conn_01x06_Pin; footprint Connector_PinHeader_2.54mm:PinHeader_1x02_P2.54mm_Vertical -> Connector_PinHeader_2.54mm:PinHeader_1x06_P2.54mm_Vertical
- J8: value Conn_01x02_Male -> Conn_01x03_Pin; footprint Connector_PinHeader_2.54mm:PinHeader_1x02_P2.54mm_Vertical -> Connector_PinHeader_2.54mm:PinHeader_1x03_P2.54mm_Vertical
- U1: value RP2040 -> Pico; footprint SnapEDA Library:QFN40P700X700X90-57N -> Frack:RPi_Pico_SMD_ohne_Debug
- U14: footprint KiCad:1043 -> Frack:Keystone_1043
- moved C38 144.8 mm to (128.6, 149.1), turned to -90 degrees
- moved C21 143.1 mm to (128.4, 145.6), turned to -90 degrees
- moved C37 140.4 mm to (130.4, 149.1), turned to 90 degrees
- moved C25 140.3 mm to (129.4, 140.1)
- moved C23 138.7 mm to (126.9, 145.6), turned to -90 degrees
- moved L11 138.7 mm to (130.4, 145.6), turned to 90 degrees
- moved L10 138.1 mm to (126.9, 145.6), turned to 90 degrees
- moved C40 137.5 mm to (130.4, 142.0), turned to 90 degrees
- moved C41 136.9 mm to (128.6, 145.6), turned to -90 degrees
- moved C39 136.8 mm to (126.9, 142.1), turned to -90 degrees
- moved C20 135.9 mm to (121.1, 140.4), turned to -90 degrees
- moved C24 135.3 mm to (119.6, 140.4), turned to -90 degrees
- moved C27 135.2 mm to (122.9, 144.6), turned to 180 degrees
- moved L8 135.0 mm to (125.9, 148.1)
- moved C26 134.8 mm to (126.4, 137.6)
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Connections:
- J1 pad 1: BAT_O -> GND
- J1 pad 3: GND -> BAT_O
- J2 pad S1: unconnected-(J2-SHIELD-PadS1) -> GND
- J2 pad S2: unconnected-(J2-SHIELD__1-PadS2) -> GND
- J2 pad S3: unconnected-(J2-SHIELD__2-PadS3) -> GND
- J2 pad S4: unconnected-(J2-SHIELD__3-PadS4) -> GND
- J6 pad 2: N_USB_BOOT -> GND
- J8 pad 1: GND -> GP8
- J8 pad 2: RESET -> GP7
- U1 pad 1: +3.3V -> UART0_TX
- U1 pad 10: +3.3V -> GP7
- U1 pad 11: unconnected-(U1-GPIO8-Pad11) -> GP8
- U1 pad 13: SEN_SCK -> GND
- U1 pad 14: SEN_MOSI -> SEN_SCK
- U1 pad 15: SEN_MISO -> SEN_MOSI
- U1 pad 16: SEN_CS -> SEN_MISO
- U1 pad 17: SEN_INT1 -> SEN_CS
- U1 pad 18: SEN_INT2 -> GND
- U1 pad 19: GND -> SEN_INT1
- U1 pad 2: SWTX -> UART0_RX
- U1 pad 20: XIN -> SEN_INT2
- U1 pad 21: XOUT -> COM_MISO
- U1 pad 22: +3.3V -> COM_CS
- U1 pad 23: +1V1 -> GND
- U1 pad 24: SWCLK -> COM_CLK
- U1 pad 25: SWD -> COM_MOSI
- U1 pad 26: RESET -> COM_DO1
- U1 pad 27: COM_MISO -> COM_DO2
- U1 pad 28: COM_CS -> GND
- U1 pad 29: COM_CLK -> unconnected-(U1-GPIO22-Pad29)
- U1 pad 3: SWRX -> GND
- U1 pad 30: COM_MOSI -> RESET
- U1 pad 31: COM_DO1 -> unconnected-(U1-GPIO26_ADC0-Pad31)
- U1 pad 32: COM_DO2 -> unconnected-(U1-GPIO27_ADC1-Pad32)
- U1 pad 33: +3.3V -> GND
- U1 pad 36: unconnected-(U1-GPIO24-Pad36) -> +3.3V
- U1 pad 37: STDLED -> unconnected-(U1-3V3_EN-Pad37)
- U1 pad 38: unconnected-(U1-GPIO26/ADC0-Pad38) -> GND
- U1 pad 39: unconnected-(U1-GPIO27/ADC1-Pad39) -> BAT_O
- U1 pad 4: LED1 -> GP2
- U1 pad 40: unconnected-(U1-GPIO28/ADC2-Pad40) -> Net-(JP1-A)
- U1 pad 5: LED2 -> GP3
- U1 pad 6: unconnected-(U1-GPIO4-Pad6) -> GP4
- U1 pad 7: unconnected-(U1-GPIO5-Pad7) -> GP5
- U1 pad 8: unconnected-(U1-GPIO6-Pad8) -> GND
- U1 pad 9: unconnected-(U1-GPIO7-Pad9) -> GP6
Routing:
- net VBUS: track 0.00 -> 63.7 mm, vias 0 -> 4
- net BAT_O: track 0.00 -> 51.3 mm, vias 0 -> 3
- net COM_MOSI: track 0.00 -> 50.9 mm, vias 0 -> 1
- net COM_DO2: track 0.00 -> 48.6 mm, vias 0 -> 1
- net DP: track 0.00 -> 47.7 mm
- net DN: track 0.00 -> 47.2 mm, vias 0 -> 2
- net COM_CLK: track 0.00 -> 45.6 mm, vias 0 -> 1
- net COM_DO1: track 0.00 -> 44.0 mm, vias 0 -> 1
- net COM_MISO: track 0.00 -> 35.2 mm, vias 0 -> 1
- net COM_CS: track 0.00 -> 32.7 mm, vias 0 -> 1
- net GND: track 0.00 -> 31.3 mm, vias 59 -> 56
- net RF_P: track 0.00 -> 17.5 mm, vias 0 -> 1
- net RF_N: track 0.00 -> 15.2 mm, vias 0 -> 1
- net BAT_P: track 0.00 -> 14.6 mm
- net +3.3V: track 0.00 -> 14.1 mm
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- added copper zone on F.Cu, net Net-(C38-Pad1)
Other:
- board size 23 x 100 mm -> 23 x 125.5 mm

Commit message: Layout Fertig
Parts:
- removed J5: Conn_01x02_Pin, Connector_PinHeader_2.54mm:PinHeader_1x02_P2.54mm_Vertical
- removed J6: Conn_01x06_Pin, Connector_PinHeader_2.54mm:PinHeader_1x06_P2.54mm_Vertical
- removed J7: Conn_01x04_Pin, Connector_PinHeader_2.54mm:PinHeader_1x04_P2.54mm_Vertical
- removed J8: Conn_01x03_Pin, Connector_PinHeader_2.54mm:PinHeader_1x03_P2.54mm_Vertical
- C33: value 1000u -> 330u; footprint Capacitor_SMD:CP_Elec_8x10.5 -> Capacitor_SMD:C_0805_2012Metric_Pad1.18x1.45mm_HandSolder
- J1, J3: value Conn_01x03_Pin -> Conn_01x06_Pin; footprint Connector_PinHeader_2.54mm:PinHeader_1x03_P2.54mm_Vertical -> Frack:PinHeader_2x03_P2.54mm_Vertical_SMD_kleiner
- J4: value Conn_01x02_Male -> Conn_01x06_Pin; footprint Connector_PinHeader_2.54mm:PinHeader_1x02_P2.54mm_Vertical -> Frack:PinHeader_2x03_P2.54mm_Vertical_SMD_kleiner
- TP1, TP2: footprint TestPoint:TestPoint_Pad_1.5x1.5mm -> Frack:TestPoint_Pad_1.5x1.5mm_small
- moved C33 84.9 mm to (130.9, 122.4), turned to -90 degrees
- moved R16 83.3 mm to (136.6, 118.7)
- moved J1 77.5 mm to (136.7, 123.7), turned to 0 degrees
- moved C18 54.8 mm to (124.7, 128.6)
- moved J4 54.3 mm to (136.2, 56.9)
- moved C19 51.5 mm to (127.7, 125.3), turned to 90 degrees
- moved U7 46.3 mm to (124.4, 125.5), turned to 0 degrees
- moved J3 29.1 mm to (123.7, 60.8)
- moved JP1 17.6 mm to (134.8, 43.6), turned to 180 degrees
- moved TP2 8.39 mm to (129.0, 67.2)
- moved TP1 7.90 mm to (130.9, 67.2)
- moved TP3 4.72 mm to (129.9, 70.5)
- moved C28 2.25 mm to (132.2, 41.6), turned to -90 degrees
- moved R1 1.90 mm to (132.2, 36.7)
- moved J2 0.33 mm to (130.0, 30.4)
Connections:
- J3 pad 1: BAT_O -> UART0_TX
- J3 pad 2: BAT_O -> UART0_RX
- J3 pad 3: +3.3V -> GP2
- J4 pad 1: GND -> RESET
- J4 pad 2: RESET -> GND
- U1 pad 31: unconnected-(U1-GPIO26_ADC0-Pad31) -> SDA
- U1 pad 32: unconnected-(U1-GPIO27_ADC1-Pad32) -> SCL
Routing:
- net BAT_O: track 51.3 -> 118.7 mm, vias 3 -> 4
- net SCL: track 0.00 -> 50.2 mm, vias 0 -> 1
- net RESET: track 0.00 -> 43.2 mm, vias 0 -> 1
- net SDA: track 0.00 -> 41.1 mm, vias 0 -> 1
- net LED_DI: track 0.00 -> 30.1 mm, vias 0 -> 1
- net +3.3V: track 14.1 -> 43.4 mm, vias 0 -> 10
- net SEN_SCK: track 0.00 -> 26.5 mm, vias 0 -> 1
- net SEN_MOSI: track 0.00 -> 23.9 mm, vias 0 -> 1
- net GP5: track 0.00 -> 22.4 mm
- net SEN_MISO: track 0.00 -> 21.6 mm
- net SEN_CS: track 0.00 -> 21.5 mm, vias 0 -> 1
- net VBUS: track 63.7 -> 43.0 mm, vias 4 -> 3
- net Net-(JP1-A): track 6.94 -> 27.0 mm, vias 0 -> 1
- net GP3: track 0.00 -> 19.8 mm, vias 0 -> 1
- net GP4: track 0.00 -> 19.0 mm
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Other:
- board text added: "DP"
- board text added: "Eberkreis Engineering GmBH ET21"
- board text added: "{dblquote}Gemeinschaft mit Büsi Herz{dblquote} ist ein offiziell eingetragenes Markenzeichen der Eberkreis Engineering Company"
- board text removed: "BOOTSEL"
- board text removed: "RESET"

Commit message: USB Differenziell
Connections:
- J1 pad 3: BAT_O -> +3.3V
- J1 pad 4: +3.3V -> BAT_O
Routing:
- net BAT_O: track 118.7 -> 122.0 mm
- net SDA: track 41.1 -> 38.1 mm
- net DP: track 37.5 -> 36.5 mm
- net SCL: track 50.2 -> 49.5 mm
- net SEN_INT2: track 16.5 -> 17.0 mm
- net GND: vias 127 -> 142

Commit message: Schema-review-1
Parts:
- removed C18, C19: 100n, Capacitor_SMD:C_0603_1608Metric_Pad1.08x0.95mm_HandSolder
- removed C28, C29: 4.7u, Capacitor_SMD:C_0603_1608Metric_Pad1.08x0.95mm_HandSolder
- removed C33: 330u, Capacitor_SMD:C_0805_2012Metric_Pad1.18x1.45mm_HandSolder
- removed R16: 470, Resistor_SMD:R_0603_1608Metric_Pad0.98x0.95mm_HandSolder
- removed U7: BMI323, SnapEDA Library:PQFN50P250X300X88-14N
- added C1: 4.7u, Capacitor_SMD:C_0603_1608Metric_Pad1.08x0.95mm_HandSolder, F.Cu at (89.8, 102.7)
- added C2: 4.7u, Capacitor_SMD:C_0603_1608Metric_Pad1.08x0.95mm_HandSolder, F.Cu at (89.8, 105.2)
- added C4: 100n, Capacitor_SMD:C_0603_1608Metric_Pad1.08x0.95mm_HandSolder, F.Cu at (78.5, 102.7)
- added C5: 100n, Capacitor_SMD:C_0603_1608Metric_Pad1.08x0.95mm_HandSolder, F.Cu at (78.5, 105.2)
- added C6: 330u, Capacitor_SMD:C_0805_2012Metric_Pad1.18x1.45mm_HandSolder, F.Cu at (83.1, 107.0)
- added J5: VBUS, Connector_PinSocket_2.54mm:PinSocket_1x01_P2.54mm_Vertical, F.Cu at (138.2, 38.5)
- added R10: 27, Resistor_SMD:R_0603_1608Metric_Pad0.98x0.95mm_HandSolder, F.Cu at (78.5, 110.2)
- added R11: 470, Resistor_SMD:R_0603_1608Metric_Pad0.98x0.95mm_HandSolder, F.Cu at (78.5, 112.7)
- added R12: 10k, Resistor_SMD:R_0603_1608Metric_Pad0.98x0.95mm_HandSolder, F.Cu at (78.3, 99.6)
- added R9: 27, Resistor_SMD:R_0603_1608Metric_Pad0.98x0.95mm_HandSolder, F.Cu at (78.5, 107.7)
- added U2: BMI160, Frack:PQFN50P250X300X88-14N, F.Cu at (83.4, 103.5)
- D2: value LED -> Blau
- D6: value LED -> Rot
- D7: value LED -> Grün
- J1, J3, J4: value Conn_01x06_Pin -> Conn_02x03_Pin
- R4: value 8k -> 8.2k
- R6, R8: value 330 -> 390
- R7: value 330 -> 430
Connections:
- net GP2 renamed GPIO2
- net GP3 renamed GPIO3
- net GP4 renamed GPIO4
- net GP5 renamed GPIO5
- net SCL renamed SCL_EXT
- net SDA renamed SDA_EXT
- D7 pad 2: BAT_O -> VBUS
- TP1 pad 1: DN -> Net-(R9-Pad1)
- TP2 pad 1: DP -> Net-(R10-Pad1)
- U1 pad 10: GP7 -> unconnected-(U1-GPIO7-Pad10)
- U1 pad 11: GP8 -> unconnected-(U1-GPIO8-Pad11)
- U1 pad 12: LED_DI -> LED_EXT
- U1 pad 9: GP6 -> unconnected-(U1-GPIO6-Pad9)
Routing:
- net LED_EXT: track 0.00 -> 30.1 mm, vias 0 -> 1
- net LED_DI: track 30.1 -> 0.00 mm, vias 1 -> 0
- net VBUS: track 43.0 -> 47.7 mm
- net GND: track 40.7 -> 39.0 mm, vias 142 -> 24
- net +3.3V: track 43.4 -> 45.2 mm, vias 10 -> 128
- added copper zone on B.Cu, net +3.3V
- added copper zone on F.Cu, net +3.3V
- added copper zone on In1.Cu, net +3.3V
- removed copper zone on B.Cu, net GND
- removed copper zone on F.Cu, net GND
- removed copper zone on In1.Cu, net GND
