File: PCB_Frackstock/MCUrp2040.kicad_sch (KiCad schematic)
At the start: 18 parts, among them J1 Conn_02x03_Pin, J2 105450-0101, J3 Conn_02x03_Pin, J4 Conn_02x03_Pin, U1 Pico, U7 BMI160

Commit message: Bauteiländerungen
Parts:
- C33: value 330u -> 100u
Changed lines of the file:
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@@
       (effects (font (size 1.27 1.27)) (justify right))
     )
-    (property "Value" "330u" (at 241.3 130.175 0)
+    (property "Value" "100u" (at 241.3 130.175 0)
       (effects (font (size 1.27 1.27)) (justify right))
     )
